File: snap.kicad_sch (KiCad schematic)
At the start: 0 parts

Commit message: worked on the schematics pt.1 and researched
Parts:
- added C1: 10uF, symbol Device:C
- added C10, C11: 30pF, symbol Device:C
- added C12, C13: 10pF, symbol Device:C
- added C2, C3, C4, C5, C7: 100nF, symbol Device:C
- added C6, C8: 1uF, symbol Device:C
- added C9: 4.7uF, symbol Device:C
- added U1: STM32U3C5RIT6, STM32U3C5RIT6:LQFP64_STM, symbol STM32U3C5RIT6:STM32U3C5RIT6
- added XTAL1: SC32S-7PF20PPM, SC32S-7PF20PPM:XTAL_SC32S-7PF20PPM_EPS, symbol SC32S-7PF20PPM:SC32S-7PF20PPM
- added Y1: ECS-80-18-23B-JTN-TR, ECS_80_18_23B_JTN_TR:XTAL_ECS-80-18-23B-JTN-TR, symbol Device:Crystal_GND24
Connections:
- new net +3V3: C1.1, C2.1, C3.1, C4.1, C5.1, C6.1, C7.1, C8.1, C9.1, U1.1 (VBAT), U1.13 (VDDA), U1.19 (VDD), U1.30 (VCAP), U1.32 (VDD), U1.48 (VDDUSB), U1.64 (VDD)
- new net GND: C1.2, C10.2, C11.2, C12.2, C13.2, C2.2, C3.2, C4.2, C5.2, C6.2, C7.2, C8.2, C9.2, U1.12 (VSSA), U1.18 (VSS), U1.31 (VSS), U1.47 (VSS), U1.63 (VSS), Y1.2 (G), Y1.4 (G)
- new net OSC32_IN: C12.1, U1.3 (PC14-OSC32_IN), XTAL1.1
- new net OSC32_OUT: C13.1, U1.4 (PC15-OSC32_OUT), XTAL1.2
- new net OSC_IN: C10.1, U1.5 (PH0-OSC_IN), Y1.1
- new net OSC_OUT: C11.1, U1.6 (PH1-OSC_OUT), Y1.3

Commit message: removed outdated schematics
Parts:
- removed C1: 10uF, symbol Device:C
- removed C10, C11: 30pF, symbol Device:C
- removed C12, C13: 10pF, symbol Device:C
- removed C2, C3, C4, C5, C7: 100nF, symbol Device:C
- removed C6, C8: 1uF, symbol Device:C
- removed C9: 4.7uF, symbol Device:C
- removed U1: STM32U3C5RIT6, STM32U3C5RIT6:LQFP64_STM, symbol STM32U3C5RIT6:STM32U3C5RIT6
- removed XTAL1: SC32S-7PF20PPM, SC32S-7PF20PPM:XTAL_SC32S-7PF20PPM_EPS, symbol SC32S-7PF20PPM:SC32S-7PF20PPM
- removed Y1: ECS-80-18-23B-JTN-TR, ECS_80_18_23B_JTN_TR:XTAL_ECS-80-18-23B-JTN-TR, symbol Device:Crystal_GND24

Commit message: added decoupling capacitors to schematic
Parts:
- added C1, C11, C13, C3, C5, C6, C7, C8, C9: 100nF, symbol Device:C
- added C10, C12, C2: 1uF, symbol Device:C
- added C4: 4.7uF, symbol Device:C
- added U1: STM32H7B3VITx, Package_QFP:LQFP-100_14x14mm_P0.5mm, symbol MCU_ST_STM32H7:STM32H7B3VITx
Connections:
- new net GND: C1.2, C10.2, C11.2, C12.2, C13.2, C2.2, C3.2, C4.2, C5.2, C6.2, C7.2, C8.2, C9.2, U1.10 (VSS), U1.19 (VSSA), U1.26 (VSS), U1.49 (VSS), U1.74 (VSS), U1.99 (VSS)
- new net VBAT: C12.1, C13.1
- new net VCAP: C1.1, U1.48 (VCAP), U1.73 (VCAP)
- new net VDDA: C10.1, C11.1, U1.21 (VDDA)
- new net VDD_MCU: C4.1, C5.1, C6.1, C7.1, C8.1, C9.1, U1.100 (VDD), U1.11 (VDD), U1.27 (VDD), U1.50 (VDD), U1.75 (VDD)
- new net VREF+: C2.1, C3.1, U1.20 (VREF+)

Commit message: actually starting to do the schematics pt.3
Parts:
- added C14, C15, C16, C17: 10pF, symbol Device:C
- added D1, D2: ESDA5V3SC5, Package_TO_SOT_SMD:SOT-23-5, symbol Power_Protection:ESDA5V3SC5
- added J1: Conn_02x07_Odd_Even, symbol Connector_Generic:Conn_02x07_Odd_Even
- added Y1: 8kHz, symbol Device:Crystal
- added Y2: 32.768kHz, symbol Device:Crystal_GND24
Connections:
- net GND: now also C14.1, C15.1, C16.1, C17.1, D1.2 (A), D2.2 (A), J1.11 (Pin_11), J1.5 (Pin_5), J1.7 (Pin_7), Y2.2 (G), Y2.4 (G)
- net OSC_IN: now reaches U1.12 (PH0)
- net OSC_IN: now also C14.2, Y1.1
- net OSC_OUT: now reaches U1.13 (PH1)
- net OSC_OUT: now also C15.2, Y1.2
- net T_SWDIO: now reaches U1.72 (PA13)
- net T_SWDIO: now also D1.5 (K), J1.4 (Pin_4)
- net T_SWCLK: now reaches U1.76 (PA14)
- net T_SWCLK: now also D1.4 (K), J1.6 (Pin_6)
- net T_JTDI: now reaches U1.77 (PA15)
- net T_JTDI: now also D1.1 (K), J1.10 (Pin_10)
- net OSC32_IN: now reaches U1.8 (PC14)
- net OSC32_IN: now also C16.2, Y2.1
- net T_SWO: now reaches U1.89 (PB3)
- net T_SWO: now also D1.3 (K), J1.8 (Pin_8)
- net OSC32_OUT: now reaches U1.9 (PC15)
- net OSC32_OUT: now also C17.2, Y2.3
- net T_NRST: now reaches U1.90 (PB4)
- net T_NRST: now also D2.5 (K), J1.12 (Pin_12)
- new net T_RX: D2.4 (K), J1.13 (Pin_13)
- new net T_TX: D2.3 (K), J1.14 (Pin_14)
- new net VDD: J1.3 (Pin_3)
- no-connect marks 0 -> 3

Commit message: actually starting to do the schematics pt.4
Parts:
- added C18, C19: 100nF, symbol Device:C
- added R1, R2: R, symbol Device:R
- added SW1, SW2: SW_DPST, symbol Switch:SW_DPST
Connections:
- net GND: now also C18.2, C19.2, R1.2, SW2.1, SW2.3
- net VDD_MCU: now also R2.1, SW1.1, SW1.3
- net NRST: now reaches U1.14 (NRST)
- net NRST: now also C19.1, R2.2, SW2.2, SW2.4
- net BOOT0: now reaches U1.94 (BOOT0)
- net BOOT0: now also C18.1, R1.1, SW1.2, SW1.4
- no-connect marks 3 -> 4
Other:
- moved on the sheet: C14, C15, C16, C17, D1, D2, J1, Y1, Y2

Commit message: actually starting to do the schematics pt.5
Parts:
- added C20: 100nF, symbol Device:C
- added D3: LED_RGBK, symbol Device:LED_RGBK
- added Q4, Q5, Q6: DMG1012T, Package_TO_SOT_SMD:SOT-523, symbol Transistor_FET:DMG1012T
- added R10, R11, R3, R4, R5, R6, R7, R8, R9: R, symbol Device:R
Connections:
- net GND: now also C20.2, Q4.2 (S), Q5.2 (S), Q6.2 (S), R3.2, R6.2, R8.2
- net VDD: now also C20.1, D3.4 (K)
- net LED_R: now reaches U1.82 (PD1)
- net LED_R: now also R4.2, R5.2, R7.2
- net LED_G: now reaches U1.83 (PD2)
- net LED_B: now reaches U1.84 (PD3)
- new net: Q6.1 (G), R7.1, R8.1
- new net: Q6.3 (D), R11.1
- new net: Q5.1 (G), R5.1, R6.1
- new net: Q5.3 (D), R10.1
- new net: D3.1 (RA), R11.2
- new net: D3.2 (GA), R10.2
- new net: D3.3 (BA), R9.2
- new net: Q4.1 (G), R3.1, R4.1
- new net: Q4.3 (D), R9.1
Other:
- moved on the sheet: C1, C10, C11, C12, C13, C14, C15, C16, C17, C18, C19, C2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
