File: snap.kicad_sch (KiCad schematic)
At the start: 43 parts, among them J1 Conn_02x07_Odd_Even, Q4 DMG1012T, Q5 DMG1012T, Q6 DMG1012T, SW1 SW_DPST, SW2 SW_DPST, U1 STM32H7B3VITx, Y1 8kHz, Y2 32.768kHz

Commit message: actually starting to do the schematics pt.6
Parts:
- removed C1, C11, C13, C18, C19, C20, C3, C5, C6, C7, C8, C9: 100nF, symbol Device:C
- removed C10, C12, C2: 1uF, symbol Device:C
- removed C14, C15, C16, C17: 10pF, symbol Device:C
- removed C4: 4.7uF, symbol Device:C
- removed D1, D2: ESDA5V3SC5, Package_TO_SOT_SMD:SOT-23-5, symbol Power_Protection:ESDA5V3SC5
- removed D3: LED_RGBK, symbol Device:LED_RGBK
- removed J1: Conn_02x07_Odd_Even, symbol Connector_Generic:Conn_02x07_Odd_Even
- removed Q4, Q5, Q6: DMG1012T, Package_TO_SOT_SMD:SOT-523, symbol Transistor_FET:DMG1012T
- removed R1, R10, R11, R2, R3, R4, R5, R6, R7, R8, R9: R, symbol Device:R
- removed SW1, SW2: SW_DPST, symbol Switch:SW_DPST
- removed U1: STM32H7B3VITx, Package_QFP:LQFP-100_14x14mm_P0.5mm, symbol MCU_ST_STM32H7:STM32H7B3VITx
- removed Y1: 8kHz, symbol Device:Crystal
- removed Y2: 32.768kHz, symbol Device:Crystal_GND24
- added R14, R15: R, symbol Device:R
- added U3: STM32H7B3VITx, Package_QFP:LQFP-100_14x14mm_P0.5mm, symbol MCU_ST_STM32H7:STM32H7B3VITx
Connections:
- net BOOT0: now also R15.1, U3.94 (BOOT0)
- net GND: now also R15.2, U3.10 (VSS), U3.19 (VSSA), U3.26 (VSS), U3.49 (VSS), U3.74 (VSS), U3.99 (VSS)
- net LED_B: now also U3.84 (PD3)
- net LED_G: now also U3.83 (PD2)
- net LED_R: now also U3.82 (PD1)
- net NRST: now also R14.2, U3.14 (NRST)
- net OSC32_IN: now also U3.8 (PC14)
- net OSC32_OUT: now also U3.9 (PC15)
- net OSC_IN: now also U3.12 (PH0)
- net OSC_OUT: now also U3.13 (PH1)
- net T_JTDI: now also U3.77 (PA15)
- net T_NRST: now also U3.90 (PB4)
- net T_SWCLK: now also U3.76 (PA14)
- net T_SWDIO: now also U3.72 (PA13)
- net T_SWO: now also U3.89 (PB3)
- net VCAP: now also U3.48 (VCAP), U3.73 (VCAP)
- net VDDA: now also U3.21 (VDDA)
- net VDD_MCU: now also R14.1, U3.100 (VDD), U3.11 (VDD), U3.27 (VDD), U3.50 (VDD), U3.75 (VDD)
- net VREF+: now also U3.20 (VREF+)
- no-connect marks 4 -> 0
Other:
- added sheet MCU peripherals (MCU_peripherals.kicad_sch)
- added sheet MCU power (MCU_power.kicad_sch)
- added sheet STLINK connector (STLINK_connector.kicad_sch)

Commit message: actually starting to do the schematics pt.7
Connections:
- net MAIN_TXD_MCU: now reaches U3.22 (PA0)
- net MAIN_RXD_MCU: now reaches U3.23 (PA1)
- net MAIN_RTS_MCU: now reaches U3.34 (PB0)
- net MAIN_CTS_MCU: now reaches U3.53 (PB14)
Other:
- added sheet comms (comms.kicad_sch)
Changed lines of the file:
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@@
+		)
+	)
+	(global_label "MAIN_RXD_MCU"
+		(shape input)
+		(at 90.17 40.64 0)
+		(fields_autoplaced yes)
+		(effects
+			(font
+				(size 1.27 1.27)
+			)
+			(justify left)
+		)
+		(property "Intersheetrefs" "${INTERSHEET_REFS}"
+			(at 107.3671 40.64 0)
+			(hide yes)
+			(show_name no)
+			(do_not_autoplace no)
+			(effects
+				(font
+					(size 1.27 1.27)
+				)
+				(justify left)
+			)
 		)
 	)
@@
 		)
 	)
+	(global_label "MAIN_RTS_MCU"
+		(shape output)
+		(at 90.17 81.28 0)
+		(fields_autoplaced yes)
+		(effects
+			(font
+				(size 1.27 1.27)
+			)
+			(justify left)
+		)
+		(property "Intersheetrefs" "${INTERSHEET_REFS}"
+			(at 107.0647 81.28 0)
+			(hide yes)
+			(show_name no)
+			(do_not_autoplace no)
+			(effects
+				(font
+					(size 1.27 1.27)
+				)
+				(justify left)
+			)
+		)
+	)
 	(global_label "T_SWO"
 		(shape input)
@@
 		)
 	)
+	(global_label "MAIN_TXD_MCU"
+		(shape output)
+		(at 90.17 38.1 0)
+		(fields_autoplaced yes)
+		(effects
+			(font
+				(size 1.27 1.27)
+			)
+			(justify left)
+		)
+		(property "Intersheetrefs" "${INTERSHEET_REFS}"
+			(at 107.0647 38.1 0)
+			(hide yes)
+			(show_name no)
+			(do_not_autoplace no)
+			(effects
+				(font
+					(size 1.27 1.27)
+				)
+				(justify left)
+			)
+		)
+	)
 	(global_label "LED_R"
 		(shape output)
@@
 				)
 				(justify right)
+			)
+		)
+	)
+	(global_label "MAIN_CTS_MCU"
+		(shape input)
+		(at 90.17 116.84 0)
+		(fields_autoplaced yes)
+		(effects
+			(font
+				(size 1.27 1.27)
+			)
+			(justify left)
+		)
+		(property "Intersheetrefs" "${INTERSHEET_REFS}"
+			(at 107.0647 116.84 0)
+			(hide yes)
+			(show_name no)
+			(do_not_autoplace no)
+			(effects
+				(font
+					(size 1.27 1.27)
+				)
+				(justify left)
 			)
 		)
@@
 	)
 	(sheet
-		(at 111.76 33.02)
+		(at 264.16 105.41)
 		(size 12.7 12.7)
 		(exclude_from_sim no)
@@
 		)
 		(property "Sheetname" "MCU power"
-			(at 111.76 32.3084 0)
+			(at 264.16 104.6984 0)
 			(show_name no)
 			(do_not_autoplace no)
@@
 		)
 		(property "Sheetfile" "MCU_power.kicad_sch"
-			(at 111.76 46.3046 0)
+			(at 264.16 118.6946 0)
 			(show_name no)
 			(do_not_autoplace no)
@@
 	)
 	(sheet
-		(at 111.76 52.07)
+		(at 264.16 124.46)
 		(size 12.7 12.7)
 		(exclude_from_sim no)
@@
 		)
 		(property "Sheetname" "MCU peripherals"
-			(at 111.76 51.3584 0)
+			(at 264.16 123.7484 0)
 			(show_name no)
 			(do_not_autoplace no)
@@
 		)
 		(property "Sheetfile" "MCU_peripherals.kicad_sch"
-			(at 111.76 65.3546 0)
+			(at 264.16 137.7446 0)
 			(show_name no)
 			(do_not_autoplace no)
@@
 	)
 	(sheet
-		(at 111.76 71.12)
+		(at 264.16 85.09)
+		(size 13.97 10.16)
+		(exclude_from_sim no)
+		(in_bom yes)
+		(on_board yes)
+		(dnp no)
+		(fields_autoplaced yes)
+		(stroke
+			(width 0.1524)
+			(type solid)
+		)
+		(fill
+			(color 0 0 0 0)
+		)
+		(property "Sheetname" "comms"
+			(at 264.16 84.3784 0)
+			(show_name no)
+			(do_not_autoplace no)
+			(effects
+				(font
+					(size 1.27 1.27)
+				)
+				(justify left bottom)
+			)
+		)
+		(property "Sheetfile" "comms.kicad_sch"
+			(at 264.16 95.8346 0)
+			(show_name no)
+			(do_not_autoplace no)
+			(effects
+				(font
+					(size 1.27 1.27)
+				)
+				(justify left top)
+			)
+		)
+		(instances
+			(project "snap"
+				(path "/30fc28b6-2d62-4a7d-b2af-6de294b3b238"
+					(page "5")
+				)
+			)
+		)
+	)
+	(sheet
+		(at 264.16 143.51)
 		(size 12.7 12.7)
 		(exclude_from_sim no)
@@
 		)
 		(property "Sheetname" "STLINK connector"
-			(at 111.76 70.4084 0)
+			(at 264.16 142.7984 0)
 			(show_name no)
 			(do_not_autoplace no)
@@
 		)
 		(property "Sheetfile" "STLINK_connector.kicad_sch"
-			(at 111.76 84.4046 0)
-			(show_name no)
-			(do_not_autoplace no)
+			(at 264.16 156.7946 0)
+			(show_name no)
+			(do_not_autoplace no)

Commit message: time to lock in for the schematic!!!
Parts:
- added AE1, AE2: 1575AT43A0040001E, symbol Device:Antenna_Chip
- added C1, C11, C13, C15, C17, C20, C21, C22, C23, C29, C3, C5, C6, C7, C8, C9: 100nF, symbol Device:C
- added C10, C12, C14, C19, C2: 1uF, symbol Device:C
- added C16, C28, C4: 4.7uF, symbol Device:C
- added C18, C30: 33pF, symbol Device:C
- added C24, C25, C26, C27: 10pF, symbol Device:C
- added C31: 100uF, symbol Device:C
- added C32, C40: 100uF, symbol Device:C_Polarized_Small
- added C33: 220nF, symbol Device:C_Small
- added C34: 47nF, symbol Device:C_Small
- added C35: 150pF, symbol Device:C_Small
- added C36: 100pF, symbol Device:C_Small
- added C37: 68pF, symbol Device:C_Small
- added C38, C42: 33pF, symbol Device:C_Small
- added C39, C43: 10pF, symbol Device:C_Small
- added C41: 100nF, symbol Device:C_Small
- added C44: 0.1uF, symbol Device:C
- added C45: 100pF, symbol Device:C
- added D1, D2: ESDA5V3SC5, Package_TO_SOT_SMD:SOT-23-5, symbol Power_Protection:ESDA5V3SC5
- added D3: CLMVC-FKA-CL1D1L71BB7C3C3, LED_SMD:LED_Cree-PLCC4_2x2mm_CW, symbol Device:LED_RGBK
- added D4, D5: ESD9B5.0ST5G, Diode_SMD:D_SOD-923, symbol Device:D_TVS_Small
- added D6, D7: LED, symbol Device:LED
- added FB1: MPZ1005A331ET, symbol Device:FerriteBead_Small
- added J1: Conn_02x07_Odd_Even, symbol Connector_Generic:Conn_02x07_Odd_Even
- added L1: 47nH, symbol Device:L
- added Q1: CSD25310Q2, Package_SON:Texas_DQK, symbol CSD25310Q2:CSD25310Q2
- added Q10, Q11, Q7, Q8, Q9: DMG1012T, Package_TO_SOT_SMD:SOT-523, symbol Transistor_FET:DMG1012T
- added R1: 39K±1%, symbol Device:R
- added R10, R3, R9: 0R, symbol Device:R
- added R11, R23: R, symbol Device:R
- added R12: 300R, symbol Device:R
- added R13: 82R, symbol Device:R
- added R16: 62R, symbol Device:R
- added R17, R19, R21: 220R, symbol Device:R
- added R18, R20, R22: 10K, symbol Device:R
- added R2: 75K±1%, symbol Device:R
- added R4: 100K, symbol Device:R
- added R5: 63.4K±1%, symbol Device:R
- added R6: 42.2K±1%, symbol Device:R
- added R7: 0R, symbol Device:R_Small
- added R8: 10R, symbol Device:R
- added SW3, SW4: SW_DPST, symbol Switch:SW_DPST
- added U1: BG95-MF, BG95:Quectel_BG95, symbol RF_GSM:BG95-MF
- added U2, U4: SGM2036S-ADJXN5G/TR, Package_TO_SOT_SMD:SOT-23-5, symbol SGM2036S-ADJXN5G_TR:SGM2036S-ADJXN5G/TR
- added U5: TXS0108EPW, Package_SO:TSSOP-20_4.4x6.5mm_P0.65mm, symbol Logic_LevelTranslator:TXS0108EPW
- added Y3: 8kHz, symbol Device:Crystal
- added Y4: 32.768kHz, symbol Device:Crystal_GND24
Connections:
- net BOOT0: now also C22.1, SW3.2, SW3.4
- net GND: now also C1.2, C10.2, C11.2, C12.2, C13.2, C14.2, C15.2, C16.2, C17.2, C18.2, C19.2, C2.2, C20.2, C21.2, C22.2, C23.2, C24.1, C25.1, C26.1, C27.1, C28.2, C29.2, C3.2, C30.2, C31.2, C32.2, C33.2, C34.2, C35.2, C36.2, C37.2, C38.2, C39.2, C4.2, C40.2, C41.2, C42.2, C43.2, C44.2, C5.2, C6.2, C7.2, C8.2, C9.2, D1.2 (A), D2.2 (A), D4.2 (A2), D5.2 (A2), J1.11 (Pin_11), J1.5 (Pin_5), J1.7 (Pin_7), Q1.3 (G), Q10.2 (S), Q11.2 (S), Q7.2 (S), Q8.2 (S), Q9.2 (S), R18.2, R2.2, R20.2, R22.2, R4.2, R6.2, SW4.1, SW4.3, U2.2 (GND), U4.2 (GND), Y4.2 (G), Y4.4 (G)
- net LED_R: now also R17.2, R19.2, R21.2
- net NRST: now also C23.1, SW4.2, SW4.4
- net OSC32_IN: now also C26.2, Y4.1
- net OSC32_OUT: now also C27.2, Y4.3
- net OSC_IN: now also C24.2, Y3.1
- net OSC_OUT: now also C25.2, Y3.2
- net T_JTDI: now also D1.1 (K), J1.10 (Pin_10)
- net T_NRST: now also D2.5 (K), J1.12 (Pin_12)
- net T_SWCLK: now also D1.4 (K), J1.6 (Pin_6)
- net T_SWDIO: now also D1.5 (K), J1.4 (Pin_4)
- net T_SWO: now also D1.3 (K), J1.8 (Pin_8)
- net VCAP: now also C1.1
- net VDDA: now also C10.1, C11.1
- net VDD_MCU: now also C4.1, C5.1, C6.1, C7.1, C8.1, C9.1, SW3.1, SW3.3
- net VREF+: now also C2.1, C3.1
- new net: D7.1 (K), R23.1
- new net: Q11.3 (D), R23.2
- new net: C19.1, C20.1, R3.1, U2.1 (VIN)
- new net: Q7.1 (G), R17.1, R18.1
- new net: R5.2, R6.1, U2.4 (BN/FB)
- new net: L1.1, R8.2
- new net: AE2.2 (PCB_Trace), C45.2, L1.2
- new net: Q8.1 (G), R19.1, R20.1
- new net: Q9.3 (D), R12.1
- new net: D3.1 (RA), R12.2
- new net: C45.1, R9.2
- new net: U1.100 (GND), U1.101 (GND), U1.102 (GND), U1.3 (GND), U1.31 (GND), U1.48 (GND), U1.50 (GND), U1.54 (GND), U1.55 (GND), U1.58 (GND), U1.59 (GND), U1.61 (GND), U1.62 (GND), U1.67 (GND), U1.68 (GND), U1.69 (GND), U1.70 (GND), U1.71 (GND), U1.72 (GND), U1.73 (GND), U1.74 (GND), U1.79 (GND), U1.80 (GND), U1.81 (GND), U1.82 (GND), U1.89 (GND), U1.90 (GND), U1.91 (GND)
- new net: U1.32 (VBAT_BB), U1.33 (VBAT_BB)
- new net: U1.52 (VBAT_RF), U1.53 (VBAT_RF)
- new net: R1.2, R2.1, U4.4 (BN/FB)
- new net: AE1.2 (PCB_Trace), R10.2
- new net: Q9.1 (G), R21.1, R22.1
- new net: Q7.3 (D), R16.1
- new net: Q10.3 (D), R11.2
- new net: D3.2 (GA), R13.2
- new net: D3.3 (BA), R16.2
- new net: D6.1 (K), R11.1
- new net: Q8.3 (D), R13.1
- new net ANTENNA_3V: C16.1, C17.1, C18.1, C44.1, R1.1, R8.1, U4.5 (VOUT)
- new net ANT_GNSS: R9.1
- new net ANT_MAIN: R10.1
- new net GNSS_EN_MCU: R4.1, U2.3 (EN)
- new net NET_STATUS: Q10.1 (G)
- new net PON_TRIG_1V8: C28.1, C29.1, C30.1, R5.1, U2.5 (VOUT)
- new net STATUS: Q11.1 (G)
- new net T_RX: D2.4 (K), J1.13 (Pin_13)
- new net T_TX: D2.3 (K), J1.14 (Pin_14)
- new net VBAT: C12.1, C13.1, C14.1, C15.1, C31.1, C32.1, C33.1, C34.1, C35.1, C36.1, C37.1, C38.1, C39.1, C40.1, C41.1, C42.1, C43.1, D4.1 (A1), D5.1 (A1), D6.2 (A), D7.2 (A), FB1.2, Q1.1 (S), Q1.2 (S), Q1.4 (D), Q1.5 (S), Q1.6 (S), Q1.7 (D), Q1.8 (S), R3.2, R7.2, U4.1 (VIN), U4.3 (EN)
- new net VBAT_BB: FB1.1
- new net VBAT_RF: R7.1
- new net VDD: C21.1, D3.4 (K), J1.3 (Pin_3)
- no-connect marks 0 -> 6
Other:
- removed sheet MCU peripherals
- removed sheet MCU power
- removed sheet STLINK connector
- removed sheet comms
- moved on the sheet: R14, R15, U3
